Commit message: 軸の向き

File: urdf/myrobot.urdf (robot description, URDF)
Before this commit: robot myrobot, 19 links, 18 joints
Joints:
- joint BL_elbow: axis 0 0 1 -> 0 0 -1
- joint BR_elbow: axis 0 0 1 -> 0 0 -1
- joint FL_shoulder: axis 0 1 0 -> 0 -1 0
- joint FR_shoulder: axis 0 1 0 -> 0 -1 0
- joint FR_wrist: axis 0 1 0 -> 0 -1 0
- joint RR_wrist: axis 0 1 0 -> 0 -1 0
